Commit message: Fix drone coverage patrol and add isolated launcher

File: urdf_parrot/parrot.gazebo.xacro (robot description, xacro)
@@ -89,5 +89,7 @@
       filename="ignition-gazebo-odometry-publisher-system"
       name="ignition::gazebo::systems::OdometryPublisher">
-      <topic>model/${gz_model_name}/odometry</topic>
+      <odom_topic>/model/${gz_model_name}/odometry</odom_topic>
+      <!-- Coverage flight needs actual z, roll and pitch feedback. -->
+      <dimensions>3</dimensions>
       <odom_publish_frequency>20</odom_publish_frequency>
       <odom_frame>${prefix}odom</odom_frame>

File: urdf_parrot/parrot.urdf.xacro (robot description, xacro)
@@ -3,4 +3,5 @@
   <xacro:arg name="prefix" default=""/>
   <xacro:property name="prefix" value="$(arg prefix)"/>
+  <xacro:arg name="camera_pitch" default="0.785398"/>
   <xacro:include filename="$(find 41068_ignition_bringup)/urdf_parrot/common_properties.urdf.xacro"/>
   <xacro:include filename="$(find 41068_ignition_bringup)/urdf_parrot/parrot.gazebo.xacro"/>
@@ -82,5 +83,5 @@
   </link>
   <joint name="${prefix}camera_joint" type="fixed">
-    <origin xyz="0.25 0.0 0.25" rpy="0 0.785398 0"/> <!-- 0.5 0.0 0.9 -->
+    <origin xyz="0.25 0.0 0.25" rpy="0 $(arg camera_pitch) 0"/>
     <parent link="${prefix}base_link"/>
     <child link="${prefix}camera_link"/>
