Commit message: vege detection refiened

File: urdf_parrot/parrot.urdf.xacro (robot description, xacro)
@@ -83,5 +83,5 @@
   </link>
   <joint name="${prefix}camera_joint" type="fixed">
-    <origin xyz="0.25 0.0 0.25" rpy="0 $(arg camera_pitch) 0"/>
+    <origin xyz="0.25 0.0 -0.15" rpy="0 $(arg camera_pitch) 0"/>
     <parent link="${prefix}base_link"/>
     <child link="${prefix}camera_link"/>

Commit message: updated lidar position

File: urdf_parrot/parrot.urdf.xacro (robot description, xacro)
@@ -64,9 +64,9 @@
     <parent link="${prefix}base_link"/>
     <child link="${prefix}base_scan"/>
-    <origin xyz="0 0 0.2" rpy="0 0 0"/>
+    <origin xyz="0 0 -0.2" rpy="0 0 0"/>
   </joint>
   <link name="${prefix}base_scan">
     <visual>
-      <origin xyz="0 0 0" rpy="0 0 0"/>
+      <origin xyz="0 0 -0.1" rpy="0 0 0"/>
       <geometry>
         <cylinder length="0.04" radius="0.09"/>
